File: DIP48-XC9572XL/DIP48-XC9572XL.sch (KiCad schematic (older format))
At the start: 10 parts, among them J1 JTAG-6, J2 Conn_01x07, U1 ADP122_3.3V_LDO_Voltage_Regul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, U2 XC9572XL-VQ64, U3 8566-VIC-IIe

Commit message: Add files via upload
Parts:
- added JP1: SJ1, Jumper:SolderJumper-3_P1.3mm_Open_RoundedPad1.0x1.5mm_NumberLabels, symbol Jumper:SolderJumper_3_Open
- added JP48: SJ48, Jumper:SolderJumper-3_P1.3mm_Open_RoundedPad1.0x1.5mm_NumberLabels, symbol Jumper:SolderJumper_3_Open
Connections:
- net +5V: now also JP1.3 (B), JP48.3 (B); no longer U3.48 (Vcc)
- net PIN_01: now also JP1.2 (C); no longer U2.58 (P58)
- new net PIN_48: JP48.2 (C), U3.48 (Vcc)
- new net PIN_4801: JP1.1 (A), JP48.1 (A), U2.58 (P58)
Changed lines of the file:
@@
 L Power2:+5V #PWR0104
 U 1 1 5F578AA2
-P 8650 2100
-F 0 "#PWR0104" H 8650 1950 50  0001 C CNN
-F 1 "+5V" H 8665 2273 50  0000 C CNN
-F 2 "" H 8650 2100 50  0001 C CNN
-F 3 "" H 8650 2100 50  0001 C CNN
-	1    8650 2100
+P 9050 1300
+F 0 "#PWR0104" H 9050 1150 50  0001 C CNN
+F 1 "+5V" H 9065 1473 50  0000 C CNN
+F 2 "" H 9050 1300 50  0001 C CNN
+F 3 "" H 9050 1300 50  0001 C CNN
+	1    9050 1300
 	1    0    0    -1
 $EndComp
@@
 	2100 4350 2000 4450
 Text Label 2100 4350 0    50   ~ 0
-PIN_01
+PIN_4801
 Wire Wire Line
 	4150 4850 4600 4850
@@
 Wire Bus Line
 	4700 1800 2000 1800
+$Comp
+L Jumper:SolderJumper_3_Open JP48
+U 1 1 5FF0211B
+P 8850 1300
+F 0 "JP48" H 8850 1505 50  0000 C CNN
+F 1 "SJ48" H 8850 1414 50  0000 C CNN
+F 2 "Jumper:SolderJumper-3_P1.3mm_Open_RoundedPad1.0x1.5mm_NumberLabels" H 8850 1300 50  0001 C CNN
+F 3 "~" H 8850 1300 50  0001 C CNN
+	1    8850 1300
+	1    0    0    -1
+$EndComp
+$Comp
+L Jumper:SolderJumper_3_Open JP1
+U 1 1 5FF03044
+P 8550 1650
+F 0 "JP1" H 8550 1855 50  0000 C CNN
+F 1 "SJ1" H 8550 1764 50  0000 C CNN
+F 2 "Jumper:SolderJumper-3_P1.3mm_Open_RoundedPad1.0x1.5mm_NumberLabels" H 8550 1650 50  0001 C CNN
+F 3 "~" H 8550 1650 50  0001 C CNN
+	1    8550 1650
+	1    0    0    -1
+$EndComp
+Entry Wire Line
+	7500 2100 7400 2200
+Text Label 7500 2100 0    50   ~ 0
+PIN_48
+Entry Wire Line
+	7500 1950 7400 2050
+Text Label 7500 1950 0    50   ~ 0
+PIN_01
+Entry Wire Line
+	7500 1800 7400 1900
+Text Label 7500 1800 0    50   ~ 0
+PIN_4801
+Wire Wire Line
+	7950 1650 7500 1650
+Entry Wire Line
+	7500 1650 7400 1750
+Text Label 7500 1650 0    50   ~ 0
+PIN_48
+Wire Wire Line
+	7500 2100 8650 2100
+Wire Wire Line
+	9050 1300 9050 1650
+Wire Wire Line
+	9050 1650 8750 1650
+Connection ~ 9050 1300
+Wire Wire Line
+	7500 1800 8350 1800
+Wire Wire Line
+	8350 1800 8350 1650
+Wire Wire Line
+	8350 1650 8350 1300
+Wire Wire Line
+	8350 1300 8650 1300
+Connection ~ 8350 1650
+Wire Wire Line
+	8550 1950 8550 1800
+Wire Wire Line
+	7500 1950 8550 1950
+Wire Wire Line
+	7950 1650 7950 1450
+Wire Wire Line
+	7950 1450 8850 1450
 Wire Bus Line
-	7400 2500 7400 6000
+	7400 1750 7400 6000
 Wire Bus Line
 	9900 1050 9900 6000
